Commit message: added robotic_arm_final.xacro

File: src/final_project_description/urdf/common_properties_final.xacro (robot description, xacro)
@@ -4,8 +4,14 @@
         <color rgba="1 0.7 0 0.8"/>
     </material>
+    <material name="red">
+        <color rgba="1 0 0 0.7"/>
+    </material>
+    <material name="blue">
+        <color rgba="0 0 1 0.7"/>
+    </material>
     <material name="second">
         <color rgba="0.3 0.3 0.25 1"/>
     </material>
-    <material name="third">
+    <material name="orange">
         <color rgba="0.8 0.3 0 1"/>
     </material>

File: src/final_project_description/urdf/mobile_base_final.xacro (robot description, xacro)
@@ -1,5 +1,5 @@
 <?xml version="1.0"?>
 <robot xmlns:xacro="http://www.ros.org/wiki/xacro">
-    <xacro:property name="base_lenght" value="0.7"/>
+    <xacro:property name="base_length" value="0.7"/>
     <xacro:property name="base_width" value="0.4"/>
     <xacro:property name="base_height" value="0.2"/>
@@ -9,5 +9,5 @@
         <visual>
             <geometry>
-                <box size="${base_lenght} ${base_width} ${base_height}" />
+                <box size="${base_length} ${base_width} ${base_height}" />
             </geometry>
             <origin xyz="0 0 ${base_height/2.0}" rpy="0 0 0"/>
@@ -16,9 +16,9 @@
         <collision>
             <geometry>
-                <box size="${base_lenght} ${base_width} ${base_height}" />
+                <box size="${base_length} ${base_width} ${base_height}" />
             </geometry>
             <origin xyz="0 0 ${base_height/2.0}" rpy="0 0 0"/>
         </collision>
-        <xacro:box_inertia m="5.0" l="${base_lenght}" w="${base_width}" h="${base_height}"
+        <xacro:box_inertia m="5.0" l="${base_length}" w="${base_width}" h="${base_height}"
                            xyz="0 0 ${base_height/2.0}" rpy="0 0 0"/>
     </link>
@@ -68,5 +68,5 @@
         <parent link="base_link"/>
         <child link="right_wheel_link"/>
-        <origin xyz="${-base_lenght/4.0} ${-(base_width + wheel_height)/2.0} 0" rpy="0 0 0"/>
+        <origin xyz="${-base_length/4.0} ${-(base_width + wheel_height)/2.0} 0" rpy="0 0 0"/>
         <axis xyz = "0 1 0"/>
     </joint>
@@ -74,5 +74,5 @@
         <parent link="base_link"/>
         <child link="left_wheel_link"/>
-        <origin xyz="${-base_lenght/4.0} ${(base_width + wheel_height)/2.0} 0" rpy="0 0 0"/>
+        <origin xyz="${-base_length/4.0} ${(base_width + wheel_height)/2.0} 0" rpy="0 0 0"/>
         <axis xyz = "0 1 0"/>
     </joint>
@@ -80,5 +80,5 @@
         <parent link="base_link"/>
         <child link="caster_wheel_link"/>
-        <origin xyz="${base_lenght/ 3.0} 0 ${-wheel_radius / 2.0}" rpy="0 0 0"/>
+        <origin xyz="${base_length/ 3.0} 0 ${-wheel_radius / 2.0}" rpy="0 0 0"/>
     </joint>
     <joint name="base_joint" type ="fixed">
